File: pcb/picox-8.kicad_pcb (KiCad board)
At the start: 2 copper layers, 287.5 x 119 mm, 131 parts, among them J1 PX-8 Expansion Port, J2 SERIAL, J3 693063010911, J4 USB_C_Receptacle_USB2.0, J5 CONN_CPLD_JTAG, J6 NTC, J7 BAT, Q1 Q_PMOS_DGS, SW1 FAILSAFE, SW2 RESET, U1 XC95144XL-TQ100, U2 MAX3222, U3 Pico_W, U5 MCP73871-2CC

Commit message: routing complete
Parts:
- added C16: 10μF, Capacitor_SMD:C_0603_1608Metric_Pad1.08x0.95mm_HandSolder, F.Cu at (189.9, 133.1)
- added C17: 10μF, Capacitor_SMD:C_0603_1608Metric_Pad1.08x0.95mm_HandSolder, F.Cu at (196.3, 133.1)
- added L1: 10µH, Inductor_THT:L_Radial_D6.0mm_P4.00mm, F.Cu at (185.1, 131.0)
- added R100: 309k, Resistor_SMD:R_0603_1608Metric_Pad0.98x0.95mm_HandSolder, F.Cu at (193.4, 129.8)
- added R99: 976k, Resistor_SMD:R_0603_1608Metric_Pad0.98x0.95mm_HandSolder, F.Cu at (196.8, 129.8)
- added U4: MCP1640Cx-xCHY, Package_TO_SOT_SMD:SOT-23-6, F.Cu at (193.2, 133.5)
- J5: value CONN_CPLD_JTAG -> CPLD_JTAG
- U2: footprint Package_SO:TSSOP-20_4.4x5mm_P0.5mm -> Package_SO:TSSOP-20_4.4x6.5mm_P0.65mm
- moved C14 64.5 mm to (202.5, 147.0)
- moved R89 31.1 mm to (291.8, 178.2), turned to -90 degrees
- moved R90 31.0 mm to (291.8, 181.7), turned to 90 degrees
- moved R92 29.1 mm to (284.2, 172.0), turned to 180 degrees
- moved R91 28.6 mm to (284.2, 170.4)
- moved C13 21.1 mm to (276.5, 179.6), turned to -90 degrees
- moved C15 10.7 mm to (274.5, 171.2), turned to 180 degrees
- moved R93 9.02 mm to (272.5, 100.3)
- moved R94 3.20 mm to (279.9, 100.3)
- moved R88 2.44 mm to (260.1, 100.2)
- moved R87 2.34 mm to (317.6, 102.0)
- moved U2 0.94 mm to (239.3, 107.7)
- moved C10 0.91 mm to (245.1, 109.4)
- moved C11 0.91 mm to (245.1, 104.9)
- moved C8 0.91 mm to (245.1, 107.9)
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Connections:
- C14 pad 1: /VB1 -> /+5V
- J1 pad 47: /VB1 -> /+5V
- J1 pad 49: /CG -> GND
- J1 pad 50: /CG -> GND
- Q1 pad 1: /VB1 -> /+5V
- U5 pad 1: /VB1 -> /VOUT
- U5 pad 20: /VB1 -> /VOUT
Routing:
- net +3.3V: track 21.6 -> 424.4 mm, vias 7 -> 15
- net /VOUT: track 0.00 -> 151.3 mm, vias 0 -> 3
- net /VBUS: track 0.00 -> 140.9 mm, vias 0 -> 2
- net Net-(J5-TMS): track 0.00 -> 92.4 mm, vias 0 -> 1
- net Net-(J5-TCK): track 0.00 -> 89.6 mm, vias 0 -> 1
- net Net-(J5-TDI): track 0.00 -> 85.1 mm, vias 0 -> 1
- net /NTC: track 0.00 -> 73.2 mm
- net Net-(J5-TDO): track 0.00 -> 71.4 mm, vias 0 -> 1
- net /+5V: track 0.00 -> 64.4 mm, vias 0 -> 3
- net /SPI: track 1.63 -> 65.4 mm, vias 0 -> 1
- net /PICO_SER_HSIN: track 0.00 -> 62.3 mm, vias 0 -> 2
- net /CHG_SEL: track 111.5 -> 170.0 mm, vias 0 -> 2
- net /CHG_PROG2: track 106.5 -> 164.7 mm, vias 0 -> 2
- net /CHG_~{PG}: track 112.7 -> 164.4 mm, vias 0 -> 2
- net /CHG_~{TE}: track 106.5 -> 157.6 mm, vias 0 -> 2
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
Commit message: pcb work
Parts:
- U4: value MCP1640Cx-xCHY -> MCP1640C
Routing:
- net /BA4: track 52.0 -> 50.6 mm
- net /BA15: track 50.3 -> 48.9 mm
- net /BA0: track 51.2 -> 49.7 mm
- net /BA2: track 48.8 -> 48.0 mm
- net /+5V: track 64.4 -> 65.1 mm
