File: pcb/picox-8.kicad_pcb (KiCad board)
At the start: 2 copper layers, 287.5 x 119 mm, 137 parts, among them J1 PX-8 Expansion Port, J2 SERIAL, J3 693063010911, J4 USB_C_Receptacle_USB2.0, J5 CPLD_JTAG, J6 NTC, J7 BAT, Q1 Q_PMOS_DGS, SW1 FAILSAFE, SW2 RESET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

Commit message: more pcb work
Parts:
- Q1: value Q_PMOS_DGS -> DMG2305UX
- U1: value XC95144XL-TQ100 -> XC95144XL
- U5: value MCP73871-2CC -> MCP73871
- moved R95 2.41 mm to (327.9, 99.1)
- moved R96 2.41 mm to (330.5, 99.1)
- moved R97 2.41 mm to (333.1, 99.1)
- moved R98 2.41 mm to (335.7, 99.1)
- moved J6 1.37 mm to (343.8, 161.8), turned to -90 degrees
- moved D1 1.31 mm to (327.9, 91.6)
- moved D2 1.31 mm to (330.5, 91.6)
- moved D3 1.31 mm to (333.1, 91.6)
- moved D4 1.31 mm to (335.7, 91.6)
Routing:
- net Net-(D3-K): track 1.91 -> 5.63 mm
- net Net-(D2-K): track 1.91 -> 5.63 mm
- net Net-(D4-K): track 1.92 -> 5.64 mm
- net Net-(D1-K): track 1.91 -> 5.63 mm
- net /LED3: track 246.6 -> 244.2 mm
- net /LED0: track 243.7 -> 241.2 mm
- net /LED2: track 245.4 -> 243.0 mm
- net /LED1: track 243.5 -> 241.2 mm
- net /NTC: track 73.2 -> 74.5 mm
- net +3.3V: track 424.4 -> 425.7 mm
Other:
- board text added: "4x100nF"

Commit message: first version sent to jlcpcb for production
Parts:
- L1: footprint Inductor_THT:L_Radial_D6.0mm_P4.00mm -> Inductor_SMD:L_1008_2520Metric_Pad1.43x2.20mm_HandSolder
- moved L1 2.33 mm to (186.5, 132.8), turned to 0 degrees
Routing:
- net /VOUT: track 151.3 -> 150.2 mm, vias 3 -> 4
- net Net-(U4-SW): track 7.34 -> 6.60 mm
