File: pcb/picox-8.kicad_sch (KiCad schematic)
At the start: 131 parts, among them J1 PX-8 Expansion Port, J2 SERIAL, J3 693063010911, J4 USB_C_Receptacle_USB2.0, J5 CONN_CPLD_JTAG, J6 NTC, J7 BAT, Q1 Q_PMOS_DGS, SW1 FAILSAFE, SW2 RESET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

Commit message: routing complete
Parts:
- added C16, C17: 10μF, Capacitor_SMD:C_0603_1608Metric_Pad1.08x0.95mm_HandSolder, symbol Device:C_Small
- added L1: 10µH, Inductor_THT:L_Radial_D6.0mm_P4.00mm, symbol Device:L_Small
- added R100: 309k, Resistor_SMD:R_0603_1608Metric_Pad0.98x0.95mm_HandSolder, symbol Device:R_Small
- added R99: 976k, Resistor_SMD:R_0603_1608Metric_Pad0.98x0.95mm_HandSolder, symbol Device:R_Small
- added U4: MCP1640Cx-xCHY, Package_TO_SOT_SMD:SOT-23-6, symbol Regulator_Switching:MCP1640Cx-xCHY
- J5: value CONN_CPLD_JTAG -> CPLD_JTAG
- U2: footprint Package_SO:TSSOP-20-1EP_4.4x6.5mm_P0.65mm_EP2.15x3.35mm -> Package_SO:TSSOP-20_4.4x6.5mm_P0.65mm
Connections:
- net CG is gone; now on net GND: J1.49 (CG), J1.50 (CG)
- net GND: now also C16.1, C17.2, R100.1, U4.2 (GND)
- net VB1 renamed +5V
- net +5V: now also C17.1, R99.2, U4.5 (V_{OUT}); no longer U5.1 (OUT), U5.20 (OUT)
- new net: L1.2, U4.1 (SW)
- new net: R100.2, R99.1, U4.4 (V_{FB})
- new net VOUT: C16.2, L1.1, U4.3 (EN), U4.6 (V_{IN}), U5.1 (OUT), U5.20 (OUT)
Other:
- moved on the sheet: C13, C14, C15, J4, J6, J7, Q1, R89, R90, R91, R92, R93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

Commit message: pcb work
Parts:
- U4: value MCP1640Cx-xCHY -> MCP1640C
Changed lines of the file:
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@@
 			)
 		)
-		(property "Value" "MCP1640Cx-xCHY"
+		(property "Value" "MCP1640C"
 			(at 168.91 220.98 0)
 			(effects

Commit message: more pcb work
Parts:
- Q1: value Q_PMOS_DGS -> DMG2305UX
- U1: value XC95144XL-TQ100 -> XC95144XL
- U5: value MCP73871-2CC -> MCP73871
Changed lines of the file:
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@@
 			)
 		)
-		(property "Value" "MCP73871-2CC"
+		(property "Value" "MCP73871"
 			(at 79.6641 218.44 0)
 			(effects
@@
 			)
 		)
-		(property "Value" "Q_PMOS_DGS"
+		(property "Value" "DMG2305UX"
 			(at 222.25 241.3 90)
 			(effects
@@
 			)
 		)
-		(property "Value" "XC95144XL-TQ100"
+		(property "Value" "XC95144XL"
 			(at 188.8841 31.75 0)
 			(effects
